Commit message: Xacro positions

File: Robotic-Arm/src/arduinobot_description/urdf/arduinobot.urdf.xacro (robot description, xacro)
@@ -74,5 +74,5 @@
         <parent link="horizontal_arm"/>
         <child link="claw_support"/>
-        <origin xyz="0 0.82 0" rpy="0 0 0"/>
+        <origin xyz="0 0.082 0" rpy="0 0 0"/>
     </joint>
     <link name="gripper_right">
